File: ATTiny48-Target-Board.kicad_sch (KiCad schematic)
At the start: 12 parts, among them J1 Conn_01x14_Pin, J2 Conn_01x14_Pin, SW1 SW_Omron_B3FS, U1 ATtiny48-P

Commit message: v1.0 ready to be paneled and sent to fab
Other:
- note removed: "BBMC-T48/T88 Bare Bones MicroController for ATtiny48 & ATtiny88"
Changed lines of the file:
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@@
     (title "ATtiny48 Breakout Board")
     (date "2023-06-13")
-    (rev "v0.4")
+    (rev "v1.0")
+    (comment 1 "Bare Bones MicroController for ATtiny48 & ATtiny88")
+    (comment 2 "BBMC-T48/T88")
   )
   (junction (at 223.52 99.06) (diameter 0) (color 0 0 0 0)
@@
     (effects (font (size 1.27 1.27)) (justify left bottom))
   )
-  (text "BBMC-T48/T88\nBare Bones MicroController for ATtiny48 & ATtiny88"
-    (at 161.29 180.34 0)
-    (effects (font (size 1.27 1.27)) (justify left bottom))
-  )

Commit message: v1.1 change hinky trace on pin 22
Parts:
- removed SW1: SW_Omron_B3FS, symbol Switch:SW_Omron_B3FS
Changed lines of the file:
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@@
   (title_block
     (title "ATtiny48 Breakout Board")
-    (date "2023-06-13")
-    (rev "v1.0")
+    (date "2023-06-14")
+    (rev "v1.1")
     (comment 1 "Bare Bones MicroController for ATtiny48 & ATtiny88")
     (comment 2 "BBMC-T48/T88")
@@
         )
       )
-    )
-  )
-  (symbol (lib_id "Switch:SW_Omron_B3FS") (at 60.96 158.75 0) (unit 1)
-    (in_bom yes) (on_board yes) (dnp no) (fields_autoplaced)
-    (property "Reference" "SW1" (at 60.96 152.4 0)
-      (effects (font (size 1.27 1.27)))
-    )
-    (property "Value" "SW_Omron_B3FS" (at 60.96 154.94 0)
-      (effects (font (size 1.27 1.27)))
-    )
-    (property "Footprint" "" (at 60.96 153.67 0)
-      (effects (font (size 1.27 1.27)) hide)
-    )
-    (property "Datasheet" "https://omronfs.omron.com/en_US/ecb/products/pdf/en-b3fs.pdf" (at 60.96 153.67 0)
-      (effects (font (size 1.27 1.27)) hide)
-    )
-    (pin "1")
-    (pin "2")
-    (instances
-      (project "ATTiny48-Target-Board"
-        (path "/4b246a24-c205-42b9-93bc-c1c2b5e80214"
-          (reference "SW1") (unit 1)
-        )
-      )
